File: docs/KiCad/Var_LIN.kicad_pcb (KiCad board)
At the start: 2 copper layers, 38.7 x 22.4 mm, 27 parts, among them J2 Conn_01x04_Pin, J3 Conn_01x04_Pin, U4 TGS_2611-E00, U5 TLIN2029ADRBRQ1, U6 LMR50410, U7 ATtiny412-SS, U8 BTS4142N

Commit message: Исправление разводки платы Ver_LIN
Parts:
- removed D7: MBRA360, Diode_SMD:D_SMA
- added D8: MBRA360, Diode_SMD:D_SMA, F.Cu at (142.7, 112.4)
- R17: footprint Resistor_SMD:R_1210_3225Metric_Pad1.30x2.65mm_HandSolder -> Resistor_SMD:R_1206_3216Metric
- moved R17 0.37 mm to (133.0, 112.4)
- moved R22 0.25 mm to (114.6, 108.8)
- moved C10 0.25 mm to (118.0, 105.8)
- moved R23 0.20 mm to (137.5, 95.6)
- moved C6 0.19 mm to (145.5, 107.3)
- moved C8 0.16 mm to (122.3, 112.2)
- moved R16 0.14 mm to (129.5, 102.7)
- moved C11 0.14 mm to (118.4, 103.9)
- moved D5 0.13 mm to (125.3, 110.3)
- moved R15 0.13 mm to (137.0, 106.3)
- moved R21 0.13 mm to (114.6, 105.4)
- moved U6 0.12 mm to (118.2, 108.3)
- moved R24 0.10 mm to (129.4, 110.2)
- moved D6 0.09 mm to (125.2, 110.2)
- moved C12 0.08 mm to (134.9, 99.4)
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Connections:
- net /Ver_LIN/+24_V renamed /+24_V
- net /Ver_LIN/+5v renamed /+5v
- net /Ver_LIN/InGas renamed /InGas
- net /Ver_LIN/LIN renamed /LIN
- net /Ver_LIN/LIN Rx renamed /LIN Rx
- net /Ver_LIN/LIN Tx renamed /LIN Tx
- net /Ver_LIN/OUT renamed /OUT
- net /Ver_LIN/Tx renamed /Tx
- net /Ver_LIN/UPDI renamed /UPDI
- J2 pad 1: /Ver_LIN/+24V -> /+24V
Routing:
- net /Ver_LIN/+24V: track 6.52 -> 0.00 mm
- net /+24V: track 0.00 -> 6.52 mm
- net Net-(U4-VH_2): track 4.01 -> 4.67 mm
Other:
- board size 38.7 x 22.4 mm -> 39 x 22.4 mm
