File: docs/KiCad/Датчик утечки газа 2026.kicad_pcb (KiCad board)
At the start: 2 copper layers, 38.7 x 22 mm, 30 parts, among them J1 Conn_01x04_Pin, J2 Conn_01x04_Pin, Q1 BC846BDW1, Q2 AO4807, U2 LMR50410, U3 ATtiny412-SS, U4 TGS_2611-E00

Commit message: Изменить выходной ключ на умный. Правки печатной платы
Parts:
- removed Q1: BC846BDW1, Package_TO_SOT_SMD:SOT-363_SC-70-6
- removed Q2: AO4807, Package_SO:SOIC-8_3.9x4.9mm_P1.27mm
- removed R11, R12: 10k, Resistor_SMD:R_0603_1608Metric
- removed R13, R14: 100, Resistor_SMD:R_0603_1608Metric
- added U1: TGS_2611-E00, Sensor_Humidity:TO180P920X780-4P, B.Cu at (137.4, 74.9)
- J2: footprint Connector_Pin:AMP SEAL 3.00mm_4p -> Connector_DIN:SSEAL_4
- R7, R8: value 100 -> 4.7k
- U4: value TGS_2611-E00 -> BTS72002EPAXUMA1; footprint Sensor:TO180P920X780-4P -> Package_TO_SOT_SMD:SOP65P600X115-15N_BTS72002EPAXUMA1; moved to F.Cu
- moved U4 19.4 mm to (155.6, 67.9)
- moved J2 13.0 mm to (155.5, 72.4), turned to 0 degrees
- moved R10 7.85 mm to (150.6, 66.7)
- moved R8 5.52 mm to (150.7, 69.9), turned to -90 degrees
- moved R9 3.71 mm to (147.1, 66.7)
- moved R7 2.23 mm to (147.2, 69.9), turned to -90 degrees
- moved R1 0.74 mm to (141.7, 74.8)
Connections:
- R10 pad 1: Net-(Q1B-B2) -> Net-(U4-DSEL)
- R7 pad 1: Net-(Q1A-B1) -> Net-(U4-IN0)
- R8 pad 1: Net-(Q1B-B2) -> Net-(U4-IN1)
- R9 pad 1: Net-(Q1A-B1) -> Net-(U4-DEN)
- U4 pad 2: /InGas -> Net-(U4-IN0)
- U4 pad 3: /+5v -> Net-(U4-DEN)
- U4 pad 4: Net-(U1-VH_2) -> unconnected-(U4-IS-Pad4)
Routing:
- net Net-(Q1A-C1): track 17.9 -> 0.00 mm, vias 2 -> 0
- net Net-(Q1B-C2): track 17.7 -> 0.00 mm, vias 2 -> 0
- net /+24_V: track 39.8 -> 24.2 mm, vias 5 -> 17
- net Net-(Q1B-B2): track 11.1 -> 0.00 mm, vias 2 -> 0
- net Net-(Q1A-B1): track 7.62 -> 0.00 mm
- net Net-(U4-IN0): track 0.00 -> 6.90 mm
- net Net-(U4-DEN): track 0.00 -> 6.02 mm, vias 0 -> 2
- net GND: track 99.4 -> 103.4 mm, vias 5 -> 2
- net Net-(U4-DSEL): track 0.00 -> 2.80 mm
- net /OUT2: track 6.17 -> 3.74 mm
- net Net-(U4-IN1): track 0.00 -> 2.38 mm
- net Net-(Q2-Pad2): track 2.08 -> 0.00 mm
- net Net-(Q2-Pad4): track 2.07 -> 0.00 mm
- net /OUT1: track 5.27 -> 3.21 mm

Commit message: Коррекция ПП. Замена выходной ключ на BTS72002
Parts:
- R2: footprint Resistor_SMD:R_1206_3216Metric -> Resistor_SMD:R_0805_2012Metric
- moved C2 6.17 mm to (135.7, 81.8)
- moved R3 5.87 mm to (137.4, 74.8)
- moved C1 5.80 mm to (133.9, 80.0)
- moved R2 0.35 mm to (149.6, 83.2), turned to 0 degrees
Routing:
- net GND: track 103.4 -> 99.9 mm, vias 2 -> 5
- net /+24_V: track 24.2 -> 22.1 mm, vias 17 -> 15
- net Net-(D2-A1): track 22.5 -> 20.5 mm
- net /UPDI: track 21.3 -> 20.8 mm
- net /InGas: track 26.6 -> 26.1 mm, vias 2 -> 1

Commit message: Коррекция схемы для драйвера BTS72002EPAXUMA1
Parts:
- U1: value TGS_2611-E00 -> TGS_2611
Connections:
- R6 pad 1: Net-(U3-PA1) -> /Tx
- R8 pad 2: Net-(U3-PA6) -> Net-(U3-PA2)
- U3 pad 2: Net-(U3-PA6) -> /InGas
- U3 pad 4: Net-(U3-PA1) -> unconnected-(U3-PA1-Pad4)
- U3 pad 5: /InGas -> Net-(U3-PA2)
Routing:
- net Net-(U3-PA2): track 0.00 -> 11.5 mm, vias 0 -> 2
- net /Tx: track 16.7 -> 26.6 mm, vias 1 -> 2
- net Net-(U3-PA6): track 9.57 -> 0.00 mm, vias 2 -> 0
- net Net-(U3-PA1): track 6.74 -> 0.00 mm
- net /InGas: track 26.1 -> 22.5 mm
Changed lines of the file:
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@@
 			(layers "F.Cu" "F.Mask" "F.Paste")
 			(roundrect_rratio 0.25)
-			(net "Net-(U3-PA6)")
+			(net "Net-(U3-PA2)")
 			(pintype "passive")
 		)
@@
 			(layers "F.Cu" "F.Mask" "F.Paste")
 			(roundrect_rratio 0.25)
-			(net "Net-(U3-PA1)")
+			(net "/Tx")
 			(pintype "passive")
 		)
@@
 			(layers "F.Cu" "F.Mask" "F.Paste")
 			(roundrect_rratio 0.25)
-			(net "Net-(U3-PA6)")
+			(net "/InGas")
 			(pinfunction "PA6_2")
 			(pintype "bidirectional")
@@
 			(layers "F.Cu" "F.Mask" "F.Paste")
 			(roundrect_rratio 0.25)
-			(net "Net-(U3-PA1)")
+			(net "unconnected-(U3-PA1-Pad4)")
 			(pinfunction "PA1_4")
 			(pintype "bidirectional")
@@
 			(layers "F.Cu" "F.Mask" "F.Paste")
 			(roundrect_rratio 0.25)
-			(net "/InGas")
+			(net "Net-(U3-PA2)")
 			(pinfunction "PA2_5")
 			(pintype "bidirectional")
@@
 			)
 		)
-		(property "Value" "TGS_2611-E00"
+		(property "Value" "TGS_2611"
 			(at -0.25 -5.375 0)
 			(layer "B.SilkS")
@@
 	)
 	(segment
-		(start 150.6585 72.254)
-		(end 150.6585 70.754)
-		(width 0.3)
-		(layer "F.Cu")
-		(net "Net-(U3-PA6)")
-	)
-	(segment
-		(start 149.2705 73.642)
-		(end 150.6585 72.254)
-		(width 0.3)
-		(layer "F.Cu")
-		(net "Net-(U3-PA6)")
-	)
-	(segment
-		(start 152.9705 77.342)
-		(end 152.9705 78.212943)
-		(width 0.3)
-		(layer "F.Cu")
-		(net "Net-(U3-PA6)")
-	)
-	(segment
-		(start 152.0005 76.372)
-		(end 152.9705 77.342)
-		(width 0.3)
-		(layer "F.Cu")
-		(net "Net-(U3-PA6)")
-	)
-	(segment
-		(start 152.0005 76.362943)
-		(end 152.0005 76.372)
-		(width 0.3)
-		(layer "F.Cu")
-		(net "Net-(U3-PA6)")
-	)
-	(via
-		(at 149.2705 73.642)
-		(size 0.6)
-		(drill 0.3)
-		(layers "F.Cu" "B.Cu")
-		(net "Net-(U3-PA6)")
-	)
-	(via
-		(at 152.0005 76.362943)
-		(size 0.6)
-		(drill 0.3)
-		(layers "F.Cu" "B.Cu")
-		(net "Net-(U3-PA6)")
-	)
-	(segment
-		(start 149.2705 73.642)
-		(end 151.991443 76.362943)
-		(width 0.3)
-		(layer "B.Cu")
-		(net "Net-(U3-PA6)")
-	)
-	(segment
-		(start 151.991443 76.362943)
-		(end 152.0005 76.362943)
-		(width 0.3)
-		(layer "B.Cu")
-		(net "Net-(U3-PA6)")
-	)
-	(segment
 		(start 139.2555 73.075)
 		(end 137.315443 71.134943)
@@
 	)
 	(segment
-		(start 155.103007 79.595435)
-		(end 155.5105 79.187942)
-		(width 0.3)
-		(layer "F.Cu")
-		(net "Net-(U3-PA1)")
-	)
-	(segment
-		(start 155.5105 79.187942)
-		(end 155.5105 78.212943)
-		(width 0.3)
-		(layer "F.Cu")
-		(net "Net-(U3-PA1)")
-	)
-	(segment
-		(start 150.2505 78.862943)
-		(end 150.2505 78.912943)
-		(width 0.3)
-		(layer "F.Cu")
-		(net "Net-(U3-PA1)")
-	)
-	(segment
-		(start 150.2505 78.912943)
-		(end 150.932992 79.595435)
-		(width 0.3)
-		(layer "F.Cu")
-		(net "Net-(U3-PA1)")
-	)
-	(segment
-		(start 150.932992 79.595435)
-		(end 155.103007 79.595435)
-		(width 0.3)
-		(layer "F.Cu")
-		(net "Net-(U3-PA1)")
-	)
-	(segment
 		(start 147.3005 78.862943)
 		(end 148.6005 78.862943)
@@
 	)
 	(segment
-		(start 155.5105 74.052943)
-		(end 155.5105 73.262943)
+		(start 136.4585 73.929)
+		(end 135.6085 73.079)
 		(width 0.3)
 		(layer "F.Cu")
@@
 	)
 	(segment
-		(start 136.4585 73.929)
-		(end 135.6085 73.079)
+		(start 152.9705 77.342)
+		(end 152.9705 78.212943)
 		(width 0.3)
 		(layer "F.Cu")
@@
 	)
 	(segment
-		(start 154.5005 75.062943)
-		(end 155.5105 74.052943)
+		(start 152.0005 76.372)
+		(end 152.9705 77.342)
 		(width 0.3)
 		(layer "F.Cu")
@@
 		(net "/InGas")
 	)
+	(segment
+		(start 152.0005 76.362943)
+		(end 152.0005 76.372)
+		(width 0.3)
+		(layer "F.Cu")
+		(net "/InGas")
+	)
 	(via
-		(at 154.5005 75.062943)
+		(at 152.0005 76.362943)
 		(size 0.6)
 		(drill 0.3)
@@
 	)
 	(segment
-		(start 151.9505 77.612943)
-		(end 154.5005 75.062943)
+		(start 151.5585 76.854)
+		(end 152.0005 76.412)
 		(width 0.3)
 		(layer "B.Cu")
@@
 	)
 	(segment
-		(start 137.622557 75.057)
-		(end 135.6555 73.089943)
+		(start 135.6555 73.089943)
+		(end 137.622557 75.057)
 		(width 0.3)
 		(layer "B.Cu")
@@
 	)
 	(segment
-		(start 144.2085 77.612943)
-		(end 141.652557 75.057)
+		(start 143.449557 76.854)
+		(end 151.5585 76.854)
+		(width 0.3)
+		(layer "B.Cu")
+		(net "/InGas")
+	)
+	(segment
+		(start 152.0005 76.412)
+		(end 152.0005 76.362943)
+		(width 0.3)
+		(layer "B.Cu")
+		(net "/InGas")
+	)
+	(segment
+		(start 151.991443 76.362943)
+		(end 152.0005 76.362943)
 		(width 0.3)
 		(layer "B.Cu")
@@
 	(segment
 		(start 141.652557 75.057)
-		(end 137.622557 75.057)
+		(end 143.449557 76.854)
 		(width 0.3)
 		(layer "B.Cu")
@@
 	)
 	(segment
-		(start 144.2085 77.612943)
-		(end 151.9505 77.612943)
+		(start 137.622557 75.057)
+		(end 141.652557 75.057)
 		(width 0.3)
 		(layer "B.Cu")
@@
 	)
 	(segment
+		(start 150.3585 77.654)
+		(end 150.3585 78.754943)
+		(width 0.3)
+		(layer "F.Cu")
+		(net "/Tx")
+	)
+	(segment
 		(start 153.0005 73.232943)
 		(end 152.9705 73.262943)
@@
 		(net "/Tx")
 	)
+	(segment
+		(start 150.2505 78.862943)
+		(end 150.2505 78.912943)
+		(width 0.3)
+		(layer "F.Cu")
+		(net "/Tx")
+	)
+	(segment
+		(start 150.3585 78.754943)
+		(end 150.2505 78.862943)
+		(width 0.3)
+		(layer "F.Cu")
+		(net "/Tx")
+	)
 	(via
 		(at 153.0005 71.504)
@@
 		(net "/Tx")
 	)
+	(via
+		(at 150.3585 77.654)
+		(size 0.6)
+		(drill 0.3)
+		(layers "F.Cu" "B.Cu")
+		(net "/Tx")
+	)
 	(segment
 		(start 139.895843 67.162943)
@@
 	)
 	(segment
+		(start 153.3505 75.982182)
+		(end 153.3585 75.990182)
+		(width 0.3)
+		(layer "B.Cu")
+		(net "/Tx")
+	)
+	(segment
+		(start 153.3585 76.454)
+		(end 152.1585 77.654)
+		(width 0.3)
+		(layer "B.Cu")
+		(net "/Tx")
+	)
+	(segment
+		(start 153.3585 75.990182)
+		(end 153.3585 76.454)
+		(width 0.3)
+		(layer "B.Cu")
+		(net "/Tx")
+	)
+	(segment
+		(start 152.1585 77.654)
+		(end 150.3585 77.654)
+		(width 0.3)
+		(layer "B.Cu")
+		(net "/Tx")
+	)
+	(segment
+		(start 153.3505 71.854)
+		(end 153.3505 75.982182)
+		(width 0.3)
+		(layer "B.Cu")
+		(net "/Tx")
+	)
+	(segment
+		(start 153.0005 71.504)
+		(end 153.3505 71.854)
+		(width 0.3)
+		(layer "B.Cu")
+		(net "/Tx")
+	)
+	(segment
 		(start 144.2369 71.504)
 		(end 139.895843 67.162943)
@@
 		(net "/Tx")
 	)
+	(segment
+		(start 155.5105 74.237942)
+		(end 155.5105 73.262943)
+		(width 0.3)
+		(layer "F.Cu")
+		(net "Net-(U3-PA2)")
+	)
+	(segment
+		(start 150.6585 72.254)
+		(end 150.6585 70.754)
+		(width 0.3)
+		(layer "F.Cu")
+		(net "Net-(U3-PA2)")
+	)
+	(segment
+		(start 149.2705 73.642)
+		(end 150.6585 72.254)
+		(width 0.3)
+		(layer "F.Cu")
+		(net "Net-(U3-PA2)")
+	)
+	(segment
+		(start 150.9585 74.954)
+		(end 154.794442 74.954)
+		(width 0.3)
+		(layer "F.Cu")
+		(net "Net-(U3-PA2)")
+	)
+	(segment
+		(start 154.794442 74.954)
+		(end 155.5105 74.237942)
+		(width 0.3)
+		(layer "F.Cu")
+		(net "Net-(U3-PA2)")
+	)
+	(via
+		(at 150.9585 74.954)
+		(size 0.6)
+		(drill 0.3)
+		(layers "F.Cu" "B.Cu")
+		(net "Net-(U3-PA2)")
+	)
+	(via
+		(at 149.2705 73.642)
+		(size 0.6)
+		(drill 0.3)
+		(layers "F.Cu" "B.Cu")
+		(net "Net-(U3-PA2)")
+	)
+	(segment
+		(start 150.5825 74.954)
+		(end 149.2705 73.642)
+		(width 0.3)
+		(layer "B.Cu")
+		(net "Net-(U3-PA2)")
+	)
+	(segment
+		(start 150.9585 74.954)
+		(end 150.5825 74.954)
+		(width 0.3)
+		(layer "B.Cu")
+		(net "Net-(U3-PA2)")
+	)
 	(zone
 		(net "GND")
@@
 		)
 		(min_thickness 0.25)
-		(fill
+		(fill yes
 			(thermal_gap 0.5)
 			(thermal_bridge_width 0.5)
