File: docs/KiCad/Датчик утечки газа 2026.kicad_sch (KiCad schematic)
At the start: 25 parts, among them J1 Conn_01x04_Pin, J2 Conn_01x04_Pin, U1 TGS_2611-E00, U2 LMR50410, U3 ATtiny412-SS, U4 BTS72002EPAXUMA1

Commit message: Обновить схемы и логику выходного ключа
Other:
- moved on the sheet: R7, R8
Changed lines of the file:
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@@
+	(wire
+		(pts
+			(xy 207.01 60.96) (xy 208.28 60.96)
+		)
+		(stroke
+			(width 0)
+			(type default)
+		)
+	)
 	(wire
 		(pts
@@
 	(wire
 		(pts
-			(xy 205.74 60.96) (xy 208.28 60.96)
+			(xy 204.47 55.88) (xy 207.01 55.88)
 		)
 		(stroke
@@
 	(wire
 		(pts
-			(xy 198.12 63.5) (xy 208.28 63.5)
+			(xy 204.47 63.5) (xy 208.28 63.5)
 		)
 		(stroke
@@
 	(wire
 		(pts
-			(xy 180.34 63.5) (xy 190.5 63.5)
+			(xy 180.34 63.5) (xy 196.85 63.5)
 		)
 		(stroke
@@
 	(wire
 		(pts
-			(xy 196.85 60.96) (xy 196.85 55.88)
-		)
-		(stroke
-			(width 0)
-			(type default)
-		)
-	)
-	(wire
-		(pts
 			(xy 58.42 113.03) (xy 58.42 129.54)
 		)
@@
 	(wire
 		(pts
-			(xy 198.12 60.96) (xy 196.85 60.96)
-		)
-		(stroke
-			(width 0)
-			(type default)
-		)
-	)
-	(wire
-		(pts
 			(xy 64.77 63.5) (xy 77.47 63.5)
 		)
@@
 		(pts
 			(xy 113.03 127) (xy 120.65 127)
+		)
+		(stroke
+			(width 0)
+			(type default)
+		)
+	)
+	(wire
+		(pts
+			(xy 207.01 55.88) (xy 207.01 60.96)
 		)
 		(stroke
@@
 	(symbol
 		(lib_id "Device:R")
-		(at 194.31 63.5 270)
+		(at 200.66 63.5 270)
 		(unit 1)
 		(body_style 1)
@@
 		(dnp no)
 		(property "Reference" "R7"
-			(at 193.04 66.04 90)
+			(at 199.39 60.706 90)
 			(show_name no)
 			(do_not_autoplace no)
@@
 		)
 		(property "Value" "4.7k"
-			(at 197.612 66.04 90)
+			(at 203.708 60.706 90)
 			(show_name no)
 			(do_not_autoplace no)
@@
 		)
 		(property "Footprint" "Resistor_SMD:R_0603_1608Metric"
-			(at 194.31 61.722 90)
+			(at 200.66 61.722 90)
 			(hide yes)
 			(show_name no)
@@
 		)
 		(property "Datasheet" ""
-			(at 194.31 63.5 0)
+			(at 200.66 63.5 0)
 			(hide yes)
 			(show_name no)
@@
 		)
 		(property "Description" "Resistor"
-			(at 194.31 63.5 0)
+			(at 200.66 63.5 0)
 			(hide yes)
 			(show_name no)
@@
 	(symbol
 		(lib_id "Device:R")
-		(at 201.93 60.96 270)
+		(at 200.66 55.88 270)
 		(unit 1)
 		(body_style 1)
@@
 		(dnp no)
 		(property "Reference" "R8"
-			(at 200.914 58.674 90)
+			(at 199.39 53.594 90)
 			(show_name no)
 			(do_not_autoplace no)
@@
 		)
 		(property "Value" "4.7k"
-			(at 205.232 58.674 90)
+			(at 203.708 53.594 90)
 			(show_name no)
 			(do_not_autoplace no)
@@
 		)
 		(property "Footprint" "Resistor_SMD:R_0603_1608Metric"
-			(at 201.93 59.182 90)
+			(at 200.66 54.102 90)
 			(hide yes)
 			(show_name no)
@@
 		)
 		(property "Datasheet" ""
-			(at 201.93 60.96 0)
+			(at 200.66 55.88 0)
 			(hide yes)
 			(show_name no)
@@
 		)
 		(property "Description" "Resistor"
-			(at 201.93 60.96 0)
-			(hide yes)
-			(show_name no)
+			(at 200.66 55.88 0)
+			(hide yes)
+			(show_name no)
